File: hardware/rpi-camera-led.kicad_sch (KiCad schematic)
At the start: 20 parts, among them J1 FFC 15P 1.0mm bottom contact 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, J2 FFC 15P 1.0mm top contact (to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, J3 Qwiic (JST SH 1.0mm), J4 SWD program header 2.54mm, Q1 AO3400A, Q2 Phototransistor, U1 CH32V003A4M6

Commit message: Route camera interposer and prepare manufacturing outputs
Update the CH32V003A4M6 pin mapping, widen and route the board around the camera lens, source the BOM, and add a DRC-gated fabrication export plus approximate assembly CAD renders.

Co-authored-by: Copilot <223556219+Copilot@users.noreply.github.com>
Parts:
- C1: DigiKey (none) -> https://www.digikey.com/en/products/result?keywords=GRM155R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; LCSC (none) -> C71687; MPN (none) -> GRM155R71A104KA01D; Manufacturer (none) -> Murata; Mouser (none) -> https://www.mouser.com/c/?q=GRM155R71A104KA01D
- C2: DigiKey (none) -> https://www.digikey.com/en/products/result?keywords=GRM155R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; LCSC (none) -> C105172; MPN (none) -> GRM155R61A105KE15D; Manufacturer (none) -> Murata; Mouser (none) -> https://www.mouser.com/c/?q=GRM155R61A105KE15D
- D1, D2: DigiKey (none) -> https://www.digikey.com/en/products/result?keywords=NCD0805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; LCSC (none) -> C110099; MPN White 0805/2835, e.g. Hongli/NationStar -> NCD0805W1; Manufacturer (none) -> Foshan NationStar Optoelectronics; Mouser (none) -> https://www.mouser.com/c/?q=NCD0805W1
- J1: DigiKey (none) -> https://www.digikey.com/en/products/result?keywords=AFA07-S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; LCSC (none) -> C262721; MPN JUSHUO AFA07-S15FCA-00 (LCSC C262721) / Amphenol SFW15R-1ST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 -> AFA07-S15FCA-00; Manufacturer (none) -> JUSHUO; Mouser (none) -> https://www.mouser.com/c/?q=AFA07-S15FCA-00
- J2: DigiKey (none) -> https://www.digikey.com/en/products/result?keywords=AFA07-S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; LCSC (none) -> C262742; MPN JUSHUO AFA07-S15ECA-00 (LCSC C262742) / Amphenol SFW15R-2ST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 -> AFA07-S15ECA-00; Manufacturer (none) -> JUSHUO; Mouser (none) -> https://www.mouser.com/c/?q=AFA07-S15ECA-00
- J3: DigiKey (none) -> https://www.digikey.com/en/products/result?keywords=SM04B-S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; LCSC (none) -> C160404; MPN JST SM04B-SRSS-TB or SH1.0-4P clone -> SM04B-SRSS-TB; Manufacturer (none) -> JST; Mouser (none) -> https://www.mouser.com/c/?q=SM04B-SRSS-TB
- J4: DigiKey (none) -> https://www.digikey.com/en/products/result?keywords=PBC03SA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; LCSC (none) -> C3333754; MPN (none) -> PBC03SAAN; Manufacturer (none) -> Sullins Connector Solutions; Mouser (none) -> https://www.mouser.com/c/?q=PBC03SAAN
- Q1: DigiKey (none) -> https://www.digikey.com/en/products/result?keywords=AO3400A; LCSC (none) -> C20917; MPN (none) -> AO3400A; Manufacturer (none) -> Alpha & Omega Semiconductor; Mouser (none) -> https://www.mouser.com/c/?q=AO3400A
- Q2: DigiKey (none) -> https://www.digikey.com/en/products/result?keywords=TEMT700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; LCSC (none) -> C499538; MPN e.g. Everlight PT17-21C/L41/TR8 -> TEMT7000X01; Manufacturer (none) -> Vishay; Mouser (none) -> https://www.mouser.com/c/?q=TEMT7000X01
- R1, R2: DigiKey (none) -> https://www.digikey.com/en/products/result?keywords=RC0402F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; LCSC (none) -> C105871; MPN (none) -> RC0402FR-074K7L; Manufacturer (none) -> Yageo; Mouser (none) -> https://www.mouser.com/c/?q=RC0402FR-074K7L
- R3, R4: value 10R -> 47R; DigiKey (none) -> https://www.digikey.com/en/products/result?keywords=RC0603F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; LCSC (none) -> C114623; MPN (none) -> RC0603FR-0747RL; Manufacturer (none) -> Yageo; Mouser (none) -> https://www.mouser.com/c/?q=RC0603FR-0747RL
- R5: DigiKey (none) -> https://www.digikey.com/en/products/result?keywords=RC0402F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; LCSC (none) -> C106232; MPN (none) -> RC0402FR-07100RL; Manufacturer (none) -> Yageo; Mouser (none) -> https://www.mouser.com/c/?q=RC0402FR-07100RL
- R8: DigiKey (none) -> https://www.digikey.com/en/products/result?keywords=RC0402F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; LCSC (none) -> C137965; MPN (none) -> RC0402FR-0710KL; Manufacturer (none) -> Yageo; Mouser (none) -> https://www.mouser.com/c/?q=RC0402FR-0710KL
- R9: DigiKey (none) -> https://www.digikey.com/en/products/result?keywords=RC0402F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; LCSC (none) -> C93943; MPN (none) -> RC0402FR-0747KL; Manufacturer (none) -> Yageo; Mouser (none) -> https://www.mouser.com/c/?q=RC0402FR-0747KL
- U1: DigiKey (none) -> https://www.digikey.com/en/products/result?keywords=CH32V00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; LCSC (none) -> C5346357; MPN WCH CH32V003A4M6 (LCSC C5346357) -> CH32V003A4M6; Manufacturer (none) -> WCH; Mouser (none) -> https://www.mouser.com/c/?q=CH32V003A4M6
Connections:
- net CAM_IO0: now also U1.12 (PA1); no longer U1.8 (PD4)
- net CAM_IO1: now also U1.13 (PA2); no longer J4.2 (Pin_2), U1.7 (PD1)
- net SCL: no longer U1.11 (PD7), U1.6 (PC7)
- net SDA: no longer U1.12 (PA1), U1.5 (PC6)
- new net SWIO: J4.2 (Pin_2), U1.7 (PD1)
Other:
- note added: "LED current is set by R3/R4 = 47R against 3V3 (about 8-15mA each for Vf=2.9-2.6V at 100% duty). Total draw comes from Pi camera 3V3 - keep the duty/current within the Pi's camera connector budget."
- note added: "R6/R7 are 10k links between the Pi and camera GPIO paths. With U1 tri-stated, the Pi signal passes through; U1 senses it on PD5/PD6 and can drive the camera on PA1/PA2. The 10k limits contention current."
- note removed: "LED current is set by R3/R4 against the 3V3 rail (about 30-40mA each with Vf=2.9V). Total draw comes from the Pi camera 3V3 supply - keep the duty/current within the Pi's camera connector budget."
- note removed: "R6/R7 (0R, DNP) are a bypass: fit them to wire the Pi's CAM_IO pins straight to the camera, e.g. when U1 is unpopulated. Left off, U1 sits in the middle -- it watches the Pi on PD5/PD6 and drives the camera on PA1/PA2. Do not fit them while U1 drives: 0R gives contention no current limit."
